File: GP2Y0D8xxZ0F.kicad_pcb (KiCad board)
At the start: 2 copper layers, 26.7 x 24.1 mm, 13 parts, among them P1 CONN_01X04, U1 GP2Y0D81xZ0F

Commit message: Moved solder Jumper for select Enable mode in Bottom Layer
Parts:
- JP1: moved to B.Cu
Routing:
- net VCC: track 53.3 -> 50.7 mm
Other:
- net class Power added: clearance 0.1524, trace_width 0.3084, via_dia 0.6858, via_drill 0.3302

Commit message: Modified trak with
Parts:
- moved P1 0.25 mm to (153.7, 100.6)
Routing:
- net GND: track 68.6 -> 70.0 mm
- net /Enable: track 16.6 -> 17.6 mm
