File: circuit/GP2Y0D8xxZ0F.sch (KiCad schematic (older format))
At the start: 9 parts, among them P1 CONN_01X04, U1 GP2Y0D81xZ0F

Commit message: First convert try and resize
Parts:
- C1, C2, C3: symbol C_Small -> Device:C_Small
- D1: symbol Led_Small -> GP2Y0D8xxZ0F-rescue:Led_Small
- JP1: symbol Jumper_NO_Small -> Device:Jumper_NO_Small
- P1: symbol CONN_01X04 -> GP2Y0D8xxZ0F-rescue:CONN_01X04
- R1, R2: symbol R -> Device:R
- U1: symbol GP2Y0D81xZ0F -> GP2Y0D8xxZ0F-rescue:GP2Y0D81xZ0F
Changed lines of the file:
@@
-EESchema Schematic File Version 2
-LIBS:power
-LIBS:device
-LIBS:transistors
-LIBS:conn
-LIBS:linear
-LIBS:regul
-LIBS:74xx
-LIBS:cmos4000
-LIBS:gp2y0d81xz0f
-LIBS:adc-dac
-LIBS:memory
-LIBS:xilinx
-LIBS:microcontrollers
-LIBS:dsp
-LIBS:microchip
-LIBS:analog_switches
-LIBS:motorola
-LIBS:texas
-LIBS:intel
-LIBS:audio
-LIBS:interface
-LIBS:digital-audio
-LIBS:philips
-LIBS:display
-LIBS:cypress
-LIBS:siliconi
-LIBS:opto
-LIBS:atmel
-LIBS:contrib
-LIBS:valves
+EESchema Schematic File Version 4
 LIBS:GP2Y0D8xxZ0F-cache
-EELAYER 25 0
+EELAYER 26 0
 EELAYER END
 $Descr A4 11693 8268
@@
 $EndDescr
 $Comp
-L GP2Y0D81xZ0F U1
+L GP2Y0D8xxZ0F-rescue:GP2Y0D81xZ0F U1
 U 1 1 56E5E3CE
 P 4600 3500
@@
 	3950 3100 4050 3100
 $Comp
-L R R1
+L Device:R R1
 U 1 1 56E5E48F
 P 3950 3750
@@
 	3950 3500 3950 3600
 Wire Wire Line
-	3950 3900 3950 4200
+	3950 3900 3950 4000
 Wire Wire Line
 	4050 4000 3950 4000
 Connection ~ 3950 4000
 $Comp
-L GND #PWR01
+L power:GND #PWR01
 U 1 1 56E5E542
 P 3950 4200
@@
 $EndComp
 $Comp
-L R R2
+L Device:R R2
 U 1 1 56E5E58C
 P 5950 3300
@@
 $EndComp
 $Comp
-L C_Small C1
+L Device:C_Small C1
 U 1 1 56E5E5BF
 P 5550 3850
@@
 $EndComp
 $Comp
-L C_Small C2
+L Device:C_Small C2
 U 1 1 56E5E620
 P 6300 3300
@@
 $EndComp
 $Comp
-L C_Small C3
+L Device:C_Small C3
 U 1 1 56E5E683
 P 6650 3300
@@
 $EndComp
 $Comp
-L Led_Small D1
+L GP2Y0D8xxZ0F-rescue:Led_Small D1
 U 1 1 56E5E6B0
 P 5950 3800
@@
 $EndComp
 Wire Wire Line
-	5150 3100 7350 3100
+	5150 3100 5250 3100
 Wire Wire Line
 	5250 3100 5250 3300
@@
 	5150 3700 5550 3700
 $Comp
-L GND #PWR02
+L power:GND #PWR02
 U 1 1 56E5E8E4
 P 6300 4200
@@
 Connection ~ 6300 3100
 Wire Wire Line
-	6300 3400 6300 4200
+	6300 3400 6300 4150
 Connection ~ 5950 4150
 Wire Wire Line
@@
 Connection ~ 6300 4150
 $Comp
-L CONN_01X04 P1
+L GP2Y0D8xxZ0F-rescue:CONN_01X04 P1
 U 1 1 56E5EB6E
 P 7550 3250
@@
 Connection ~ 6650 4150
 $Comp
-L Jumper_NO_Small JP1
+L Device:Jumper_NO_Small JP1
 U 1 1 56E5EEA5
 P 5500 3300
@@
 	5550 3950 5550 4150
 Wire Wire Line
-	5550 4150 7300 4150
+	5550 4150 5950 4150
 Wire Wire Line
 	5550 3700 5550 3750
 $Comp
-L VCC #PWR03
+L power:VCC #PWR03
 U 1 1 56E5F591
 P 5950 3000
@@
 $EndComp
 Wire Wire Line
-	5950 3000 5950 3150
+	5950 3000 5950 3100
+Wire Wire Line
+	3950 4000 3950 4200
+Wire Wire Line
+	5250 3100 5500 3100
+Wire Wire Line
+	5950 3100 5950 3150
+Wire Wire Line
+	5950 3100 6300 3100
+Wire Wire Line
+	6300 3100 6650 3100
+Wire Wire Line
+	5950 4150 6300 4150
+Wire Wire Line
+	6300 4150 6300 4200
+Wire Wire Line
+	6300 4150 6650 4150
+Wire Wire Line
+	6650 3100 7350 3100
+Wire Wire Line
+	6650 4150 7300 4150
+Wire Wire Line
+	5500 3100 5950 3100
 $EndSCHEMATC
