File: circuit/GP2Y0D8xxZ0F.kicad_pcb (KiCad board)
At the start: 2 copper layers, 25 x 25 mm, 13 parts, among them P1 CONN_01X04, U1 GP2Y0D81xZ0F

Commit message: Generated gerber and drill file
Routing:
- net VCC: track 48.5 -> 51.1 mm
Other:
- board text added: "@bobboteck"
- board text added: "Settorezero.com"
Changed lines of the file:
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@@
-(kicad_pcb (version 20171130) (host pcbnew "(5.0.2)-1")
+(kicad_pcb (version 20171130) (host pcbnew "(5.0.1)-4")
   (general
     (thickness 1.6002)
-    (drawings 10)
-    (tracks 65)
+    (drawings 16)
+    (tracks 66)
     (zones 0)
     (modules 13)
@@
   )
   (setup
-    (last_trace_width 0.3048)
+    (last_trace_width 0.1524)
     (user_trace_width 0.1524)
     (user_trace_width 0.3048)
@@
     (visible_elements 7FFFFF7F)
     (pcbplotparams
-      (layerselection 0x010f0_80000001)
+      (layerselection 0x010fc_ffffffff)
       (usegerberextensions true)
       (usegerberattributes false)
@@
   (module GP2Y0D81xZ0F:GP2Y0D81xZ0F (layer F.Cu)
     (at 81 84)
-    (fp_text reference U1 (at -5.665 -6.35) (layer F.SilkS)
+    (fp_text reference U1 (at 5.5 -6.35 90) (layer F.SilkS)
       (effects (font (size 1 1) (thickness 0.15)))
     )
@@
     (tags "resistor 0201")
     (attr smd)
-    (fp_text reference JP1 (at 0 1.7) (layer B.SilkS)
+    (fp_text reference JP1 (at 0 -2.5 90) (layer B.SilkS)
       (effects (font (size 1 1) (thickness 0.15)) (justify mirror))
     )
@@
       (rotate (xyz 0 0 0))
     )
+  )
+  (gr_text @bobboteck (at 80 82 90) (layer B.SilkS)
+    (effects (font (size 1 1) (thickness 0.25)) (justify mirror))
+  )
+  (gr_text Settorezero.com (at 74.5 83.5 90) (layer F.SilkS)
+    (effects (font (size 1 1) (thickness 0.25)))
   )
   (gr_arc (start 71 78.5) (end 71 76) (angle -90) (layer Edge.Cuts) (width 0.15))
@@
   (segment (start 85.75 78) (end 86 78.25) (width 0.3048) (layer B.Cu) (net 3))
   (segment (start 86 78.25) (end 86 82.5) (width 0.3048) (layer B.Cu) (net 3))
+  (segment (start 91.5 86.087) (end 91.5 83.49874) (width 0.1524) (layer F.Cu) (net 3))
   (segment (start 91.5 90.5) (end 91.5 90.913) (width 0.3048) (layer F.Cu) (net 4))
   (segment (start 88 87) (end 91.5 90.5) (width 0.3048) (layer F.Cu) (net 4))
